Commit message: can_be_run

File: assets/models/urdf/omni copy.urdf (robot description, URDF)
Before this commit: robot phantom_omni, 7 links, 6 joints
Joints:
- joint elbow: axis 1 0 0 -> 0 1 0; limit lower=-0.81 upper=1.25 effort=5 velocity=100 -> lower=0.0 upper=1.5 effort=5 velocity=100; origin xyz=0.0075 .134 0 rpy=-1.5 0 0 -> xyz=0.134 -0.0075 0 rpy=0 1.5708 0
- joint pitch: axis 1 0 0 -> 0 1 0; origin xyz=0 0.0525 0 rpy=0 0 0 -> xyz=0.0525 0 0 rpy=0 1 0
- joint roll: axis 0 1 0 -> 1 0 0; origin xyz=0 -0.023 0 rpy=3.14159 3.14159 0 -> xyz=-0.023 0 0 rpy=0 0 3.14159
- joint shoulder: axis 1 0 0 -> 0 1 0; origin xyz=-0.0075 0 0.035 rpy=0 0 0 -> xyz=0 0.0075 0.035 rpy=0 0 0
- joint yaw: axis 0 1 0 -> 1 0 0; origin xyz=0 0.08 0 -> xyz=0.08 0 0

File: assets/models/urdf/omni_2 copy.urdf (robot description, URDF)
Before this commit: robot phantom_omni, 7 links, 6 joints
Links:
- link lower_arm: mass 0.0001 -> 0.08
- link stylus: mass 0.2 -> 0.03
- link torso: mass 0.0001 -> 0.14
- link upper_arm: mass 0.0001 -> 0.10
Joints:
- joint elbow: axis 1 0 0 -> 0 1 0; limit lower=-0.81 upper=1.25 effort=5 velocity=100 -> lower=-0.7854 upper=1.5 effort=5 velocity=100; origin xyz=0.0075 .134 0 rpy=-1.5 0 0 -> xyz=-0.134 0.0075 0 rpy=0 3.14159 0
- joint pitch: axis 1 0 0 -> 0 1 0; limit lower=-0.5 upper=2.5 effort=5 velocity=100 -> lower=0 upper=2.5 effort=5 velocity=100; origin xyz=0 0.0525 0 rpy=0 0 0 -> xyz=0 0 -0.0525 rpy=3.14159 0 0
- joint roll: axis 0 1 0 -> 0 0 1; origin xyz=0 -0.023 0 rpy=3.14159 3.14159 0 -> xyz=0 0 -0.023 rpy=3.14159 0 0
- joint shoulder: axis 1 0 0 -> 0 1 0; origin xyz=-0.0075 0 0.035 rpy=0 0 0 -> xyz=0 0.0075 0.035 rpy=0 0 3.14159
- joint yaw: axis 0 1 0 -> 0 0 1; origin xyz=0 0.08 0 -> xyz=0 0 0.08 rpy=3.14159 0 0

File: assets/models/urdf/omni_2.urdf (robot description, URDF)
Before this commit: robot phantom_omni, 7 links, 6 joints
Joints:
- joint elbow: axis 1 0 0 -> 0 1 0; limit lower=-0.81 upper=1.25 effort=5 velocity=100 -> lower=-0.7854 upper=1.5 effort=5 velocity=100; origin xyz=0.0075 .134 0 rpy=-1.5 0 0 -> xyz=-0.134 0.0075 0 rpy=0 3.14159 0
- joint pitch: axis 1 0 0 -> 0 1 0; limit lower=-0.5 upper=2.5 effort=5 velocity=100 -> lower=0 upper=2.5 effort=5 velocity=100; origin xyz=0 0.0525 0 rpy=0 0 0 -> xyz=0 0 -0.0525 rpy=3.14159 0 0
- joint roll: axis 0 1 0 -> 0 0 1; origin xyz=0 -0.023 0 rpy=3.14159 3.14159 0 -> xyz=0 0 -0.023 rpy=3.14159 0 0
- joint shoulder: axis 1 0 0 -> 0 1 0; origin xyz=-0.0075 0 0.035 rpy=0 0 0 -> xyz=0 0.0075 0.035 rpy=0 0 3.14159
- joint yaw: axis 0 1 0 -> 0 0 1; origin xyz=0 0.08 0 -> xyz=0 0 0.08 rpy=3.14159 0 0
